Commit message: Update control for cooperative system

File: urdf_model/ur5e.urdf (robot description, URDF)
Before this commit: robot ur5e, 11 links, 10 joints
Links:
- added link gripper_link
Joints:
- added joint tool0-gripper_link_fixed_joint: type fixed, parent tool0, child gripper_link, origin xyz=0 0.0 0.155 rpy=0 0 0

File: urdf_model/ur5e_left.urdf (robot description, URDF)
Before this commit: robot ur5e, 11 links, 10 joints
Links:
- added link gripper_link
Joints:
- added joint tool0-gripper_link_fixed_joint: type fixed, parent tool0, child gripper_link, origin xyz=0 0.0 0.0 rpy=0 0 0
- joint world_joint: origin xyz=0.0 -1.1 0.0 rpy=0.0 0.0 -3.14159265359 -> xyz=0.1029 -1.0467 -0.0910 rpy=0 0 -3.14159265359

File: urdf_model/ur5e_right.urdf (robot description, URDF)
Before this commit: robot ur5e, 11 links, 10 joints
Links:
- added link gripper_link
Joints:
- added joint tool0-gripper_link_fixed_joint: type fixed, parent tool0, child gripper_link, origin xyz=0 0.0 0.0 rpy=0 0 0
