Commit message: Gripper and object link added

File: urdf_model/ur5e_fc.urdf (robot description, URDF)
Before this commit: robot ur5e, 12 links, 11 joints
Links:
- added link gripper
- added link obj
Joints:
- added joint gripper-obj_fixed_joint: type fixed, parent gripper, child obj, origin xyz=0 0 0.05325 rpy=0 0 0
- added joint tool0-gripper_fixed_joint: type fixed, parent tool0, child gripper, origin xyz=0 0 0.182697 rpy=0 0 0
