Commit message: Add cooperative calculation for orient and pose, also for force

File: urdf_model/ur5e_left.urdf (robot description, URDF)
Before this commit: robot ur5e, 11 links, 10 joints
Joints:
- joint base_link-base_fixed_joint: origin xyz=0 0 0 rpy=0 0 -3.14159265359 -> xyz=0 0 0 rpy=0 0 0.0
- joint world_joint: origin xyz=0.0 0.0 0.0 rpy=0.0 -110.0 0.0 -> xyz=0.0 -1.1 0.0 rpy=0.0 0.0 -3.14159265359

File: urdf_model/ur5e_right.urdf (robot description, URDF)
Before this commit: robot ur5e, 11 links, 10 joints
Joints:
- joint world_joint: origin xyz=0.0 0.0 0.0 rpy=0.0 0.0 0.0 -> xyz=0.0 0.0 0.0 rpy=0.0 0.0 -3.14159265359

Commit message: Add controller, add full pose/orient controller

File: urdf_model/ur5e_left.urdf (robot description, URDF)
Before this commit: robot ur5e, 12 links, 11 joints
Joints:
- joint tool0-gripper_link_fixed_joint: origin xyz=0 0.0 0.0 rpy=0 0 0 -> xyz=0 0.0 0.155 rpy=0 0 0
- joint world_joint: origin xyz=0.1029 -1.0467 -0.0910 rpy=0 0 -3.14159265359 -> xyz=0.1029 -1.0467 -0.0910 rpy=-0.0043 -0.0153 -3.0625

Commit message: Add smart command for p2p move

File: urdf_model/ur5e_left.urdf (robot description, URDF)
Before this commit: robot ur5e, 12 links, 11 joints
Joints:
- joint world_joint: origin xyz=0.1029 -1.0467 -0.0910 rpy=-0.0043 -0.0153 -3.0625 -> xyz=0.1029 -1.0467 -0.0810 rpy=-0.0043 -0.0153 -3.0625

Commit message: Create executer and json reader

File: urdf_model/ur5e_left.urdf (robot description, URDF)
Before this commit: robot ur5e, 12 links, 11 joints
Joints:
- joint world_joint: origin xyz=0.1029 -1.0467 -0.0810 rpy=-0.0043 -0.0153 -3.0625 -> xyz=0.1029 -1.0460 -0.0683 rpy=-0.0012 -0.0082 -3.0759

Commit message: Recalibrate URs in 449

File: urdf_model/ur5e_left.urdf (robot description, URDF)
Before this commit: robot ur5e, 12 links, 11 joints
Joints:
- joint world_joint: origin xyz=0.1029 -1.0460 -0.0683 rpy=-0.0012 -0.0082 -3.0759 -> xyz=0.0 0.0 0.0 rpy=0.0 0.0 -3.14159265359

File: urdf_model/ur5e_right.urdf (robot description, URDF)
Before this commit: robot ur5e, 12 links, 11 joints
Joints:
- joint world_joint: origin xyz=0.0 0.0 0.0 rpy=0.0 0.0 -3.14159265359 -> xyz=0.825 0.028 0.0683 rpy=-0.000 -0.000 -3.04159265359
